File: RP2040_MCU.kicad_pcb (KiCad board)
At the start: 2 copper layers, 0 parts

Commit message: Routing in Progress
Parts:
- added C1: 22pF, Capacitor_SMD:C_0603_1608Metric, F.Cu at (128.9, 61.3)
- added C10: 1uF, Capacitor_SMD:C_0603_1608Metric, F.Cu at (143.8, 46.7)
- added C11: 1uF, Capacitor_SMD:C_0603_1608Metric, F.Cu at (146.1, 49.6)
- added C12: 1uF, Capacitor_SMD:C_0603_1608Metric, F.Cu at (146.3, 52.2)
- added C13: 1uF, Capacitor_SMD:C_0603_1608Metric, F.Cu at (132.4, 52.0)
- added C14: 1uF, Capacitor_SMD:C_0603_1608Metric, F.Cu at (139.7, 63.4)
- added C15: 1uF, Capacitor_SMD:C_0603_1608Metric, F.Cu at (148.1, 56.9)
- added C16: 1uF, Capacitor_SMD:C_0603_1608Metric, F.Cu at (131.9, 56.6)
- added C17: 1uF, Capacitor_SMD:C_0603_1608Metric, F.Cu at (145.7, 34.0)
- added C18: 1uF, Capacitor_SMD:C_0603_1608Metric, F.Cu at (146.4, 41.8)
- added C2: 22pF, Capacitor_SMD:C_0603_1608Metric, F.Cu at (129.0, 63.3)
- added C3: 10uF, Capacitor_SMD:C_0603_1608Metric, F.Cu at (145.7, 31.0)
- added C4: 1uF, Capacitor_SMD:C_0603_1608Metric, F.Cu at (130.0, 36.1)
- added C5: 1uF, Capacitor_SMD:C_0603_1608Metric, F.Cu at (134.8, 47.1)
- added C6: 1uF, Capacitor_SMD:C_0603_1608Metric, F.Cu at (142.0, 63.3)
- added C7: 1uF, Capacitor_SMD:C_0603_1608Metric, F.Cu at (141.6, 46.7)
- added C8: 1uF, Capacitor_SMD:C_0603_1608Metric, F.Cu at (139.1, 47.0)
- added C9: 1uF, Capacitor_SMD:C_0603_1608Metric, F.Cu at (137.1, 47.0)
- added J1: USB_C_Receptacle_USB2.0, Connector_USB:USB_C_Receptacle_HRO_TYPE-C-31-M-12, F.Cu at (139.2, 23.9)
- added J2: Conn_01x18, Connector_PinSocket_2.54mm:PinSocket_1x18_P2.54mm_Vertical, F.Cu at (124.8, 21.7)
- added J3: Conn_01x18, Connector_PinSocket_2.54mm:PinSocket_1x18_P2.54mm_Vertical, F.Cu at (156.2, 21.6)
- added R1: 1k, Resistor_SMD:R_0603_1608Metric, F.Cu at (130.7, 31.6)
- added R2: 5k1, Resistor_SMD:R_0603_1608Metric, F.Cu at (142.3, 31.6)
- added R3: 5k1, Resistor_SMD:R_0603_1608Metric, F.Cu at (136.1, 31.6)
- added R4: 1k, Resistor_SMD:R_0603_1608Metric, F.Cu at (137.4, 63.4)
- added R5: 1k, Resistor_SMD:R_0603_1608Metric, F.Cu at (148.0, 47.0)
- added R6: 27, Resistor_SMD:R_0603_1608Metric, F.Cu at (138.9, 43.0)
- added R7: 27, Resistor_SMD:R_0603_1608Metric, F.Cu at (141.9, 43.0)
- added R8: 1k, Resistor_SMD:R_0603_1608Metric, F.Cu at (148.0, 44.3)
- added SW1: SW_Push, Button_Switch_SMD:SW_Push_SPST_NO_Alps_SKRK, F.Cu at (130.7, 26.4)
- added SW2: SW_Push, Button_Switch_SMD:SW_Push_SPST_NO_Alps_SKRK, F.Cu at (147.7, 26.5)
- added U1: W25Q128JVS, Package_SO:SOIC-8_5.23x5.23mm_P1.27mm, F.Cu at (134.3, 39.1)
- added U2: USBLC6-2SC6, Package_TO_SOT_SMD:SOT-23-6, F.Cu at (140.4, 37.2)
- added U3: RP2040, Package_DFN_QFN:QFN-56-1EP_7x7mm_P0.4mm_EP3.2x3.2mm, F.Cu at (139.2, 55.4)
- added U4: XC6206PxxxMR, Package_TO_SOT_SMD:SOT-23, F.Cu at (146.6, 37.8)
- added Y1: Crystal_GND23, Crystal:Crystal_SMD_3225-4Pin_3.2x2.5mm, F.Cu at (132.8, 62.7)
Routing:
- net +3V3: track 0.00 -> 75.2 mm, vias 0 -> 3
- net /GPIO28: track 0.00 -> 36.8 mm
- net /GPIO29: track 0.00 -> 36.5 mm
- net /GPIO0: track 0.00 -> 36.1 mm
- net /GPIO27: track 0.00 -> 35.3 mm
- net +5V: track 0.00 -> 34.9 mm, vias 0 -> 2
- net /GPIO26: track 0.00 -> 34.4 mm
- net /GPIO1: track 0.00 -> 34.1 mm
- net QSPI_SS: track 0.00 -> 32.2 mm
- net /GPIO2: track 0.00 -> 32.1 mm
- net /GPIO25: track 0.00 -> 31.2 mm
- net /GPIO24: track 0.00 -> 30.8 mm
- net /GPIO3: track 0.00 -> 30.0 mm
- net /GPIO4: track 0.00 -> 28.0 mm
- net QSPI_SD1: track 0.00 -> 27.7 mm
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