File: RP2040_MCU.kicad_sch (KiCad schematic)
At the start: 1 part, among them U1 RP2040

Commit message: Finished Schematic of RP2040 MCU
Parts:
- added C1, C2: 22pF, Capacitor_SMD:C_0402_1005Metric, symbol Device:C
- added C10, C11, C12, C13, C14, C15, C16, C17, C4, C5, C6, C7, C8, C9: 1uF, Capacitor_SMD:C_0402_1005Metric, symbol Device:C
- added C3: 10uF, Capacitor_SMD:C_0402_1005Metric, symbol Device:C
- added J1: USB_C_Receptacle_USB2.0, Connector_USB:USB_C_Receptacle_HRO_TYPE-C-31-M-12, symbol Connector:USB_C_Receptacle_USB2.0
- added J2, J3: Conn_01x18, Connector_PinSocket_2.54mm:PinSocket_1x18_P2.54mm_Vertical, symbol Connector_Generic:Conn_01x18
- added R1, R4, R5, R8: 1k, Resistor_SMD:R_0402_1005Metric, symbol Device:R
- added R2, R3: 5k1, Resistor_SMD:R_0402_1005Metric, symbol Device:R
- added R6, R7: 27, Resistor_SMD:R_0402_1005Metric, symbol Device:R
- added SW1, SW2: SW_Push, Button_Switch_SMD:SW_Push_1P1T_NO_CK_KSC6xxJ, symbol Switch:SW_Push
- added U1: W25Q128JVS, Package_SO:SOIC-8_5.23x5.23mm_P1.27mm, symbol Memory_Flash:W25Q128JVS
- added U2: USBLC6-2SC6, Package_TO_SOT_SMD:SOT-23-6, symbol Power_Protection:USBLC6-2SC6
- added U3: XC6206PxxxMR, Package_TO_SOT_SMD:SOT-23, symbol Regulator_Linear:XC6206PxxxMR
- added Y1: Crystal_GND23, Crystal:Crystal_SMD_3225-4Pin_3.2x2.5mm, symbol Device:Crystal_GND23
- U4: renamed from U1; LCSC (none) -> C2040
Connections:
- net +3V3: now reaches U4.1 (IOVDD), U4.10 (IOVDD), U4.22 (IOVDD), U4.33 (IOVDD), U4.42 (IOVDD), U4.49 (IOVDD)
- net +3V3: now also U4.43 (ADC_AVDD), U4.44 (VREG_IN), U4.48 (USB_VDD), C10.2, C11.2, C12.2, C13.2, C14.2, C15.2, C16.2, C17.2, C4.2, C9.2, J2.1 (Pin_1), J3.1 (Pin_1), R5.2, U1.8 (VCC), U3.2 (VO)
- net GPIO8: now reaches U4.11 (GPIO8)
- net GPIO8: now also J2.10 (Pin_10)
- net GPIO9: now reaches U4.12 (GPIO9)
- net GPIO9: now also J2.11 (Pin_11)
- net GPIO10: now reaches U4.13 (GPIO10)
- net GPIO10: now also J2.12 (Pin_12)
- net GPIO11: now reaches U4.14 (GPIO11)
- net GPIO11: now also J2.13 (Pin_13)
- net GPIO12: now reaches U4.15 (GPIO12)
- net GPIO12: now also J2.14 (Pin_14)
- net GPIO13: now reaches U4.16 (GPIO13)
- net GPIO13: now also J2.15 (Pin_15)
- net GPIO14: now reaches U4.17 (GPIO14)
- net GPIO14: now also J2.16 (Pin_16)
- net GPIO15: now reaches U4.18 (GPIO15)
- net GPIO15: now also J2.17 (Pin_17)
- net GND: now reaches U4.19 (TESTEN)
- net GND: now also U4.57 (GND), C1.2, C10.1, C11.1, C12.1, C13.1, C14.1, C15.1, C16.1, C17.1, C2.2, C3.1, C4.1, C5.1, C6.1, C7.1, C8.1, C9.1, J1.A1 (GND), J1.A12 (GND), J1.B1 (GND), J1.B12 (GND), J2.18 (Pin_18), J3.18 (Pin_18), R2.1, R3.1, SW1.1, SW2.1, U1.4 (GND), U2.2 (GND), U3.1 (GND), Y1.2, Y1.3
- net GPIO0: now reaches U4.2 (GPIO0)
- net GPIO0: now also J2.2 (Pin_2)
- net XIN: now reaches U4.20 (XIN)
- net XIN: now also C1.1, Y1.4
- net XOUT: now reaches U4.21 (XOUT)
- net XOUT: now also R4.2
- net +1V1: now reaches U4.23 (DVDD), U4.50 (DVDD)
- net +1V1: now also U4.45 (VREG_VOUT), C5.2, C7.2, C8.2
- net SWCLK: now reaches U4.24 (SWCLK)
- net SWCLK: now also J3.17 (Pin_17)
- net SWD: now reaches U4.25 (SWD)
- net SWD: now also J3.16 (Pin_16)
- net RESET: now reaches U4.26 (RUN)
- net RESET: now also R5.1, R8.2
- net GPIO16: now reaches U4.27 (GPIO16)
- net GPIO16: now also J3.2 (Pin_2)
- net GPIO17: now reaches U4.28 (GPIO17)
- net GPIO17: now also J3.3 (Pin_3)
- net GPIO18: now reaches U4.29 (GPIO18)
- net GPIO18: now also J3.4 (Pin_4)
- net GPIO1: now reaches U4.3 (GPIO1)
- net GPIO1: now also J2.3 (Pin_3)
- net GPIO19: now reaches U4.30 (GPIO19)
- net GPIO19: now also J3.5 (Pin_5)
- net GPIO20: now reaches U4.31 (GPIO20)
- net GPIO20: now also J3.6 (Pin_6)
- net GPIO21: now reaches U4.32 (GPIO21)
- net GPIO21: now also J3.7 (Pin_7)
- net GPIO22: now reaches U4.34 (GPIO22)
- net GPIO22: now also J3.8 (Pin_8)
- net GPIO23: now reaches U4.35 (GPIO23)
- net GPIO23: now also J3.9 (Pin_9)
- net GPIO24: now reaches U4.36 (GPIO24)
- net GPIO24: now also J3.10 (Pin_10)
- net GPIO25: now reaches U4.37 (GPIO25)
- net GPIO25: now also J3.11 (Pin_11)
- net GPIO26: now reaches U4.38 (GPIO26_ADC0)
- net GPIO26: now also J3.12 (Pin_12)
- net GPIO27: now reaches U4.39 (GPIO27_ADC1)
- net GPIO27: now also J3.13 (Pin_13)
- net GPIO2: now reaches U4.4 (GPIO2)
- net GPIO2: now also J2.4 (Pin_4)
- net GPIO28: now reaches U4.40 (GPIO28_ADC2)
- net GPIO28: now also J3.14 (Pin_14)
- net GPIO29: now reaches U4.41 (GPIO29_ADC3)
- net GPIO29: now also J3.15 (Pin_15)
- net at U4.46 (USB_DM): now also R6.2
- net at U4.47 (USB_DP): now also R7.2
- net GPIO3: now reaches U4.5 (GPIO3)
- net GPIO3: now also J2.5 (Pin_5)
- net QSPI_SD3: now reaches U4.51 (QSPI_SD3)
- net QSPI_SD3: now also U1.7 (IO3)
- net QSPI_SCLK: now reaches U4.52 (QSPI_SCLK)
- net QSPI_SCLK: now also U1.6 (CLK)
- net QSPI_SD0: now reaches U4.53 (QSPI_SD0)
- net QSPI_SD0: now also U1.5 (DI(IO0))
- net QSPI_SD2: now reaches U4.54 (QSPI_SD2)
- net QSPI_SD2: now also U1.3 (IO2)
- net QSPI_SD1: now reaches U4.55 (QSPI_SD1)
- net QSPI_SD1: now also U1.2 (DO(IO1))
- net QSPI_SS: now reaches U4.56 (QSPI_SS)
- net QSPI_SS: now also R1.2, U1.1 (~{CS})
- net GPIO4: now reaches U4.6 (GPIO4)
- net GPIO4: now also J2.6 (Pin_6)
- net GPIO5: now reaches U4.7 (GPIO5)
- net GPIO5: now also J2.7 (Pin_7)
- net GPIO6: now reaches U4.8 (GPIO6)
- net GPIO6: now also J2.8 (Pin_8)
- net GPIO7: now reaches U4.9 (GPIO7)
- net GPIO7: now also J2.9 (Pin_9)
- new net: C2.1, R4.1, Y1.1
- new net: J1.A5 (CC1), R2.2
- new net: R8.1, SW2.2
- new net: J1.B5 (CC2), R3.2
- new net: R1.1, SW1.2
- new net +5V: C3.2, C6.2, J1.A4 (VBUS), J1.A9 (VBUS), J1.B4 (VBUS), J1.B9 (VBUS), U2.5 (VBUS), U3.3 (VI)
- new net USB_D+: J1.A6 (D+), J1.B6 (D+), U2.6 (I/O1)
- new net USB_D-: J1.A7 (D-), J1.B7 (D-), U2.4 (I/O2)
- new net USB_DM: R6.1, U2.3 (I/O2)
- new net USB_DP: R7.1, U2.1 (I/O1)
- no-connect marks 0 -> 3
Other:
- moved on the sheet: U4

Commit message: Routing in Progress
Parts:
- removed C17: 1uF, Capacitor_SMD:C_0402_1005Metric, symbol Device:C
- removed R6: 27, Resistor_SMD:R_0402_1005Metric, symbol Device:R
- added C18, C6: 1uF, Capacitor_SMD:C_0603_1608Metric, symbol Device:C
- added R7: 27, Resistor_SMD:R_0603_1608Metric, symbol Device:R
- C1, C10, C11, C12, C13, C14, C15, C16, C2, C3, C5, C7, C8, C9: footprint Capacitor_SMD:C_0402_1005Metric -> Capacitor_SMD:C_0603_1608Metric
- C17: renamed from C6; footprint Capacitor_SMD:C_0402_1005Metric -> Capacitor_SMD:C_0603_1608Metric
- C4: footprint Capacitor_SMD:C_0402_1005Metric -> Capacitor_SMD:C_0603_1608Metric; LCSC (none) -> C52923
- R1, R2, R3, R4, R5, R8: footprint Resistor_SMD:R_0402_1005Metric -> Resistor_SMD:R_0603_1608Metric
- R6: renamed from R7; footprint Resistor_SMD:R_0402_1005Metric -> Resistor_SMD:R_0603_1608Metric
- SW1: footprint Button_Switch_SMD:SW_Push_1P1T_NO_CK_KSC6xxJ -> Button_Switch_SMD:SW_Push_SPST_NO_Alps_SKRK
- SW2: footprint Button_Switch_SMD:SW_Push_1P1T_NO_CK_KSC6xxJ -> Button_Switch_SMD:SW_Push_SPST_NO_Alps_SKRK; LCSC (none) -> C720477
- renumbered U4 to U3, U3 to U4
Connections:
- net +1V1: now also C6.2; no longer C8.2
- net +3V3: now also C8.2, C18.2
- net GND: now also R3.2, C18.1, C6.1; no longer R3.1
- net GPIO16: now also J3.15 (Pin_15); no longer J3.2 (Pin_2)
- net GPIO17: now also J3.14 (Pin_14); no longer J3.3 (Pin_3)
- net GPIO18: now also J3.13 (Pin_13); no longer J3.4 (Pin_4)
- net GPIO19: now also J3.12 (Pin_12); no longer J3.5 (Pin_5)
- net GPIO20: now also J3.11 (Pin_11); no longer J3.6 (Pin_6)
- net GPIO21: now also J3.10 (Pin_10); no longer J3.7 (Pin_7)
- net GPIO22: now also J3.9 (Pin_9); no longer J3.8 (Pin_8)
- net GPIO23: now also J3.8 (Pin_8); no longer J3.9 (Pin_9)
- net GPIO24: now also J3.7 (Pin_7); no longer J3.10 (Pin_10)
- net GPIO25: now also J3.6 (Pin_6); no longer J3.11 (Pin_11)
- net GPIO26: now also J3.5 (Pin_5); no longer J3.12 (Pin_12)
- net GPIO27: now also J3.4 (Pin_4); no longer J3.13 (Pin_13)
- net GPIO28: now also J3.3 (Pin_3); no longer J3.14 (Pin_14)
- net GPIO29: now also J3.2 (Pin_2); no longer J3.15 (Pin_15)
- net RESET: now also R8.1, SW2.2; no longer R5.1, R8.2, U3.26 (RUN)
- net DN: now reaches U3.46 (USB_DM)
- net DN: now also R7.2
- net DP: now reaches R6.2, U3.47 (USB_DP)
- net CrysOut: now reaches C2.1, R4.1, Y1.1
- net CC1: now reaches J1.A5 (CC1), R2.2
- net CC2: now reaches J1.B5 (CC2)
- net CC2: now also R3.1; no longer R3.2
- net BOOT: now reaches R1.1, SW1.2
- net USB_D+ renamed D+
- net USB_D- renamed D-
- net USB_DM renamed USB_DN
- net USB_DN: now also R7.1
- new net RUN: R5.1, R8.2, U3.26 (RUN)
Other:
- moved on the sheet: C1, C17, R2, SW1, U4, Y1
